File: Blocky_Uno/Blocky_Uno.brd (EAGLE design)
At the start: 68.7 x 53.5 mm, 52 parts, among them J1 10118193-0001LF, U1 1117-3.3V, U2 CH340T, U4 ATmega328mu, X1 12MHz, X2 16MHz

Commit message: Update Blocky Uno
Parts:
- removed J1: 10118193-0001LF, Seeed-Connector -2016:MICRO-USB5+6P-SMD-0.65-B
- removed U$2: (no value), Logo:OSHW_FILLX200_NOTEXT
- added U$9: MICRO-USB, My-Eagle-Lib:MICRO-USB
- U$4: device Logo:LOGO_SILK -> Anata-Symbols:BLOCKY_LOGO
- moved U$4 26.2 mm to (24.5, 14.9)
Connections:
- removed net N$12: F1.1, J1.1, VCC.T
- new net VBUS: F1.1, U$9.1, VCC.T
- net GND: now also U$9.5, U$9.GND1, U$9.GND2; no longer J1.5, J1.S1, J1.S2, J1.S3, J1.S4, J1.S5, J1.S6
- net USB_D+: now also U$9.3; no longer J1.3
- net USB_D-: now also U$9.2; no longer J1.2
Routing:
- net N$12: track 11.2 -> 0.00 mm, vias 2 -> 0
- net VBUS: track 0.00 -> 9.87 mm, vias 0 -> 2
- added copper zone on layer 1, net VBUS
- removed copper zone on layer 1, net N$12
Other:
- outline, holes or cut-outs redrawn
- board text added: "Blocky Uno"
- board text removed: "Seeeduino Lotus"
- board text removed: "by Seeed Studio"
- board text removed: "v1.0 05/16/2014"
- board text removed: "www.seeedstudio.com"
