File: Blocky_Mini_Ultra/Blocky_Mini_Ultra.brd (EAGLE design)
At the start: 57.8 x 25.8 mm, 42 parts, among them IC3 MCP1703CB, J1 2P-2.0-90D-SMD, J2 10118193-0001LF, U1 MCP73831, X1 16 MHz, X4 12MHz

Commit message: Update schematic
Routing:
- added copper zone on layer 1, net GND
- added copper zone on layer 16, net GND
Changed lines of the file:
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@@
 <setting verticaltext="up"/>
 </settings>
-<grid distance="10" unitdist="mil" unit="mil" style="lines" multiple="1" display="no" altdistance="0.1" altunitdist="mm" altunit="mm"/>
+<grid distance="10" unitdist="mil" unit="mil" style="dots" multiple="1" display="yes" altdistance="0.1" altunitdist="mm" altunit="mm"/>
 <layers>
 <layer number="1" name="Top" color="4" fill="1" visible="yes" active="yes"/>
@@
 <wire x1="16.256" y1="15.8496" x2="16.256" y2="17.5768" width="0.381" layer="1"/>
 <wire x1="15.526203125" y1="18.306596875" x2="15.24" y2="18.5928" width="0.381" layer="1"/>
+<polygon width="0.254" layer="1">
+<vertex x="51.054" y="25.908"/>
+<vertex x="51.054" y="0"/>
+<vertex x="-6.604" y="0"/>
+<vertex x="-6.604" y="25.908"/>
+</polygon>
+<polygon width="0.254" layer="16">
+<vertex x="-6.604" y="25.908"/>
+<vertex x="-6.604" y="0"/>
+<vertex x="51.054" y="0"/>
+<vertex x="51.054" y="25.908"/>
+</polygon>
 </signal>
 <signal name="RST">

Commit message: Replace usb for mini ultra
Parts:
- removed J2: 10118193-0001LF, Seeed-Connector -2016:MICRO-USB5+6P-SMD-0.65-B
- added U$5: MICRO-USB, My-Eagle-Lib:MICRO-USB
- moved RST 0.51 mm to (-3.30, 2.41)
Connections:
- net GND: now also U$5.5, U$5.GND1, U$5.GND2; no longer J2.5, J2.S1, J2.S2, J2.S3, J2.S4, J2.S5, J2.S6
- net USB_D+: now also U$5.3; no longer J2.3
- net USB_D-: now also U$5.2; no longer J2.2
- net VBUS: now also U$5.1; no longer J2.1
Routing:
- net GND: track 209.8 -> 213.6 mm
- net VBUS: track 21.3 -> 22.2 mm

Commit message: Correct error for Ultra Mini
Parts:
- moved SJ1 6.86 mm to (53.3, 14.1)
- moved SJ2 6.86 mm to (53.2, 10.8)
- moved SJ3 6.86 mm to (53.2, 8.51)
- moved U$1 6.86 mm to (53.6, 17.6)
- moved U$2 6.86 mm to (56.6, 4.70)
- moved W25X40CLSNIG-ND 6.86 mm to (51.1, 8.64)
- moved C1 6.86 mm to (24.7, 15.9)
- moved C12 6.86 mm to (27.6, 11.6)
- moved C2 6.86 mm to (21.9, 19.5)
- moved C3 6.86 mm to (31.1, 15.5)
- moved C5 6.86 mm to (9.53, 12.3)
- moved C8 6.86 mm to (24.4, 11.6)
- moved C9 6.86 mm to (27.2, 19.4)
- moved R1 6.86 mm to (24.1, 19.5)
- moved R3 6.86 mm to (27.6, 15.8)
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Routing:
- net GND: track 213.6 -> 203.5 mm
- net DIO2: track 5.27 -> 2.22 mm
- net DIO1: track 4.93 -> 2.89 mm
- net RA02_RST: track 4.85 -> 3.02 mm
- net VCC: track 105.8 -> 105.1 mm
