File: Blocky_Node/Blocky_Node.brd (EAGLE design)
At the start: 48.2 x 54.8 mm, 52 parts, among them J3 DIP Grove, J4 DIP Grove, J5 DIP Grove, J6 DIP Grove, J7 DIP Grove, J8 DIP Grove, K1 button 311020045, K2 button 311020045, Q3 S8050, Q6 S8050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

Commit message: Update Blocky Node
Parts:
- CHG: device microbuilder:CHIPLED_0805_NOOUTLINE -> microbuilder:CHIPLED_0603
- moved U$15 16.4 mm to (34.5, 18.2)
- moved C6 0.57 mm to (25.9, 11.2)
Connections:
- removed net EN: U2.3
- net POW: now also U2.3
Routing:
- net D+: track 25.9 -> 19.0 mm, vias 0 -> 2
- net D-: track 22.7 -> 17.2 mm, vias 0 -> 2
- net POW: track 9.58 -> 14.6 mm
- net GND: track 127.1 -> 128.6 mm, vias 73 -> 74
- net GND_SW: track 188.6 -> 187.8 mm, vias 6 -> 8
- net GPIO2: track 114.2 -> 114.8 mm
- net GPIO13: track 31.3 -> 31.9 mm
Other:
- board text added: "Blocky NODE WiFi"
- board text removed: "Blocky NODE"
