File: Blocky_Node/Blocky_Node.sch (EAGLE design)
At the start: 51 parts, among them J3 DIP Grove, J4 DIP Grove, J5 DIP Grove, J6 DIP Grove, J7 DIP Grove, J8 DIP Grove, K1 button 311020045, K2 button 311020045, Q3 S8050, Q6 S8050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

Commit message: Update Blocky Node
Parts:
- CHG: device microbuilder:LED0805_NOOUTLINE -> microbuilder:LED0603
Connections:
- removed net EN: U2.EN
- net POW: now also U2.EN
