File: Blocky_Uno_ESP32/Blocky_Uno_ESP32.sch (EAGLE design)
At the start: 53 parts, among them Q2 S8050, Q3 DMG3415U, Q6 S8050, U1 ESP-WROOM-32NARROW, U2 AP2112-3.3, U5 MCP73831T-2ACI/OT, U6 CH340C, X1 JSTPH

Commit message: Fix error with GND trace
Parts:
- removed LOGO1: REVISION, SparkFun-Aesthetics:REVISION
- removed LOGO3: OSHW-LOGOS, SparkFun-Aesthetics:OSHW-LOGOS
- FRAME1: value FRAME-LETTER -> (none); device SparkFun-Aesthetics:FRAME-LETTER -> SparkFun-Aesthetics:FRAME-LETTERNO_PACKAGE
Other:
- note removed: "Bruce"
- note removed: "Wangcf"
Changed lines of the file:
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@@
 <part name="A3" library="Connector" deviceset="TWIG-4P-2.0" device="-2.0"/>
 <part name="I2C.." library="Connector" deviceset="TWIG-4P-2.0" device="-2.0"/>
-<part name="U$1" library="moudle" deviceset="SEEEDSTUDIO_SCH_FRAME" device=""/>
 <part name="A2" library="Connector" deviceset="TWIG-4P-2.0" device="-2.0"/>
 <part name="GND" library="Discrete" deviceset="PAD-TEST-POINT" device="'4545'"/>
@@
 <part name="U3" library="moudle" deviceset="ARDUINO-38P" device=""/>
 <part name="U$9" library="My-Eagle-Lib" deviceset="MICRO-USB" device=""/>
-<part name="FRAME1" library="SparkFun-Aesthetics" deviceset="FRAME-LETTER" device=""/>
 <part name="U1" library="SparkFun-RF" deviceset="ESP-WROOM-32" device="NARROW"/>
 <part name="R1" library="SparkFun-Resistors" deviceset="10KOHM" device="-0603-1/10W-1%" value="10k"/>
@@
 <part name="C7" library="SparkFun-Capacitors" deviceset="0.1UF" device="-0603-25V-(+80/-20%)" value="0.1uF"/>
 <part name="C9" library="SparkFun-Capacitors" deviceset="0.1UF" device="-0603-25V-(+80/-20%)" value="0.1uF"/>
-<part name="LOGO3" library="SparkFun-Aesthetics" deviceset="OSHW-LOGO" device="S" value="OSHW-LOGOS"/>
-<part name="LOGO1" library="SparkFun-Aesthetics" deviceset="REVISION" device=""/>
 <part name="FD3" library="SparkFun-Aesthetics" deviceset="FIDUCIAL" device="1X2"/>
 <part name="FD1" library="SparkFun-Aesthetics" deviceset="FIDUCIAL" device="1X2"/>
@@
 <part name="R36" library="SparkFun-Resistors" deviceset="0.27OHM" device="-0603-1/10W-1%" value="10K"/>
 <part name="R37" library="SparkFun-Resistors" deviceset="0.27OHM" device="-0603-1/10W-1%" value="10K"/>
+<part name="FRAME1" library="SparkFun-Aesthetics" deviceset="FRAME-LETTER" device="NO_PACKAGE"/>
 </parts>
 <sheets>
 <sheet>
 <plain>
-<text x="190.5" y="11.43" size="1.778" layer="97" ratio="10">Wangcf</text>
-<text x="224.79" y="11.43" size="1.778" layer="97" ratio="10">Bruce</text>
 <text x="535.94" y="138.43" size="1.905" layer="97" font="vector">Boot Mode Configuration
 Pin        Default     Boot   Download
@@
 <attribute name="VALUE" x="389.89" y="6.35" size="1.27" layer="96" rot="R270"/>
 </instance>
-<instance part="U$1" gate="G$1" x="0" y="0" smashed="yes">
-<attribute name="DRAWING_NAME" x="191.77" y="19.05" size="2.032" layer="94" font="vector" ratio="10"/>
-<attribute name="SHEET" x="246.38" y="5.08" size="1.778" layer="94" font="vector" ratio="10"/>
-<attribute name="LAST_DATE_TIME" x="186.69" y="5.08" size="1.27" layer="94" ratio="10"/>
-</instance>
 <instance part="A2" gate="G$1" x="392.43" y="31.75" smashed="yes" rot="R180">
 <attribute name="NAME" x="393.7" y="26.67" size="1.27" layer="95" rot="R180"/>
@@
 <attribute name="VALUE" x="384.81" y="157.734" size="1.778" layer="96"/>
 </instance>
-<instance part="FRAME1" gate="G$1" x="281.94" y="-5.08" smashed="yes"/>
-<instance part="FRAME1" gate="V" x="429.26" y="-5.08" smashed="yes">
-<attribute name="LAST_DATE_TIME" x="441.96" y="-3.81" size="2.54" layer="94" font="vector"/>
-<attribute name="SHEET" x="515.62" y="-3.81" size="2.54" layer="94" font="vector"/>
-<attribute name="DRAWING_NAME" x="444.754" y="12.7" size="2.7432" layer="94" font="vector"/>
-</instance>
 <instance part="U1" gate="G$1" x="317.5" y="45.72" smashed="yes">
 <attribute name="NAME" x="302.26" y="81.534" size="1.778" layer="95"/>
@@
 <attribute name="VALUE" x="296.164" y="66.421" size="1.778" layer="96" font="vector"/>
 </instance>
-<instance part="LOGO3" gate="G$1" x="515.62" y="26.67" smashed="yes"/>
-<instance part="LOGO1" gate="G$1" x="430.784" y="1.524" smashed="yes"/>
 <instance part="FD3" gate="G$1" x="528.32" y="15.24" smashed="yes"/>
 <instance part="FD1" gate="G$1" x="525.78" y="15.24" smashed="yes"/>
@@
 <attribute name="VALUE" x="497.332" y="155.956" size="1.778" layer="96" font="vector" align="top-center"/>
 </instance>
+<instance part="FRAME1" gate="G$1" x="281.94" y="-5.08" smashed="yes"/>
+<instance part="FRAME1" gate="V" x="429.26" y="-5.08" smashed="yes">
+<attribute name="LAST_DATE_TIME" x="441.96" y="-3.81" size="2.54" layer="94" font="vector"/>
+<attribute name="SHEET" x="515.62" y="-3.81" size="2.54" layer="94" font="vector"/>
+<attribute name="DRAWING_NAME" x="444.754" y="12.7" size="2.7432" layer="94" font="vector"/>
+</instance>
 </instances>
