File: Blocky_Uno/v2/Blocky_Uno_v2.sch (EAGLE design)
At the start: 40 parts, among them U1 1117-3.3V, U4 ATmega328p-au, Y1 16MHZ, Y2 12MHz

Commit message: Update frame info
Other:
- note removed: "Bruce"
- note removed: "Wangcf"
