File: Blocky_Uno_ESP32/v1.1/Blocky_ESP32.brd (EAGLE design)
At the start: 68.7 x 53.5 mm, 51 parts, among them Q2 S8050, Q3 DMG3415U, Q6 S8050, U1 ESP-WROOM-32, U2 AP2112-3.3, U5 MCP73831T-2ACI/OT, U6 CH340C, X1 JSTPH

Commit message: Update pinout for Uno ESP32
Connections:
- net IO25: now also D1.1; no longer D1.2
- net IO26: now also D1.2; no longer D1.1
Routing:
- net GND: track 488.1 -> 489.1 mm
- net IO26: track 88.9 -> 88.0 mm
- net IO25: track 99.0 -> 98.4 mm, vias 2 -> 3
Changed lines of the file:
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@@
 <text x="49.403" y="16.002" size="0.889" layer="21" ratio="11">GND</text>
 <text x="49.403" y="14.097" size="0.889" layer="21" ratio="11">VCC</text>
-<text x="49.403" y="12.192" size="0.889" layer="21" ratio="11">25</text>
-<text x="49.403" y="10.287" size="0.889" layer="21" ratio="11">26</text>
+<text x="49.403" y="12.192" size="0.889" layer="21" ratio="11">26</text>
+<text x="49.403" y="10.287" size="0.889" layer="21" ratio="11">25</text>
 <text x="59.182" y="16.002" size="0.889" layer="21" ratio="11">GND</text>
 <text x="59.182" y="14.097" size="0.889" layer="21" ratio="11">VCC</text>
@@
 <contactref element="A2" pad="4"/>
 <polygon width="0.2032" layer="16" isolate="0.254" rank="6">
-<vertex x="-0.127" y="0"/>
+<vertex x="-0.254" y="0"/>
 <vertex x="68.58" y="0"/>
 <vertex x="68.58" y="53.34"/>
-<vertex x="-0.127" y="53.34"/>
+<vertex x="-0.254" y="53.34"/>
 </polygon>
 <polygon width="0.2032" layer="1" isolate="0.254" rank="6">
-<vertex x="-0.127" y="0"/>
+<vertex x="-0.254" y="0"/>
 <vertex x="68.58" y="0"/>
 <vertex x="68.58" y="53.34"/>
-<vertex x="-0.127" y="53.34"/>
+<vertex x="-0.254" y="53.34"/>
 </polygon>
 <contactref element="U3" pad="15"/>
@@
 <wire x1="21.0185" y1="8.7249" x2="21.8948" y2="9.6012" width="0.1524" layer="1"/>
 <wire x1="19.8374" y1="8.7249" x2="21.0185" y2="8.7249" width="0.1524" layer="1"/>
-<wire x1="19.558" y1="8.8392" x2="19.75485" y2="8.64235" width="0.1524" layer="1"/>
+<wire x1="19.558" y1="8.8392" x2="19.7104" y2="8.6868" width="0.1524" layer="1"/>
+<wire x1="19.7104" y1="8.6868" x2="19.75485" y2="8.64235" width="0.1524" layer="1"/>
 <wire x1="19.558" y1="9.9361" x2="19.558" y2="8.8392" width="0.1524" layer="1"/>
 <wire x1="22.5806" y1="9.6012" x2="22.606" y2="9.613" width="0.1524" layer="1"/>
@@
 <wire x1="17.4498" y1="7.9375" x2="17.4498" y2="6.6675" width="0.1524" layer="1"/>
 <wire x1="15.5448" y1="11.2776" x2="15.5448" y2="15.7353" width="0.1524" layer="1"/>
-<wire x1="19.7104" y1="8.5979" x2="19.8374" y2="8.7249" width="0.1524" layer="1"/>
+<wire x1="19.7104" y1="8.5979" x2="19.78025" y2="8.66775" width="0.1524" layer="1"/>
+<wire x1="19.78025" y1="8.66775" x2="19.8374" y2="8.7249" width="0.1524" layer="1"/>
 <wire x1="10.5664" y1="9.7409" x2="10.5664" y2="7.5565" width="0.1524" layer="1"/>
 <wire x1="10.5664" y1="9.7409" x2="11.3411" y2="10.5156" width="0.1524" layer="1"/>
@@
 <wire x1="14.605" y1="44.069" x2="14.986" y2="44.069" width="0.2032" layer="1"/>
 <wire x1="14.986" y1="44.069" x2="15.494" y2="43.561" width="0.2032" layer="1"/>
-<wire x1="25.54" y1="31.9405" x2="25.54" y2="31.877" width="0" layer="19" extent="1-1"/>
-<wire x1="19.75485" y1="8.64235" x2="19.7104" y2="8.5979" width="0" layer="19" extent="1-1"/>
-<wire x1="13.589" y1="3.544" x2="13.6017" y2="3.4671" width="0" layer="19" extent="1-1"/>
-<wire x1="7.366" y1="3.517" x2="7.2898" y2="3.556" width="0" layer="19" extent="1-1"/>
-<wire x1="15.24" y1="37.592" x2="15.2908" y2="38.1381" width="0" layer="19" extent="1-1"/>
+<wire x1="13.6017" y1="3.4671" x2="13.589" y2="3.544" width="0.1524" layer="1"/>
+<wire x1="7.2898" y1="3.556" x2="7.366" y2="3.517" width="0.1524" layer="1"/>
+<wire x1="19.7358" y1="8.7122" x2="19.7104" y2="8.6868" width="0.1524" layer="1"/>
+<wire x1="19.7358" y1="8.7122" x2="19.78025" y2="8.66775" width="0.1524" layer="1"/>
+<wire x1="25.5143" y1="31.9151" x2="25.54" y2="31.877" width="0.1524" layer="1"/>
+<wire x1="25.5143" y1="31.9151" x2="25.54" y2="31.9405" width="0.1524" layer="1"/>
+<wire x1="15.2908" y1="38.1381" x2="15.2908" y2="37.6047" width="0.1524" layer="1"/>
+<wire x1="15.2908" y1="37.6047" x2="15.24" y2="37.592" width="0.1524" layer="1"/>
 </signal>
 <signal name="AREF">
@@
 <via x="40.9194" y="38.7096" extent="1-16" drill="0.3048"/>
 <via x="52.959" y="31.1658" extent="1-16" drill="0.3048"/>
+<wire x1="13.9573" y1="46.5836" x2="13.89" y2="46.592" width="0.1524" layer="1"/>
 <wire x1="13.9573" y1="46.5836" x2="14.0208" y2="46.5836" width="0.1524" layer="1"/>
-<wire x1="13.9573" y1="46.5836" x2="13.89" y2="46.592" width="0" layer="19" extent="1-1"/>
 </signal>
 <signal name="SCL_22">
@@
 <contactref element="U1" pad="10"/>
 <contactref element="U3" pad="4"/>
-<contactref element="D1" pad="2"/>
 <wire x1="19.1135" y1="27.9019" x2="19.4818" y2="27.5336" width="0.1524" layer="1"/>
 <wire x1="22.7838" y1="27.5336" x2="19.4818" y2="27.5336" width="0.1524" layer="1"/>
@@
 <wire x1="33.9598" y1="16.4719" x2="33.9598" y2="19.4691" width="0.1524" layer="1"/>
 <wire x1="34.9631" y1="15.4686" x2="33.9598" y2="16.4719" width="0.1524" layer="1"/>
-<wire x1="43.307" y1="15.4686" x2="34.9631" y2="15.4686" width="0.1524" layer="1"/>
+<wire x1="38.227" y1="15.4686" x2="34.9631" y2="15.4686" width="0.1524" layer="1"/>
 <wire x1="55.9181" y1="49.4284" x2="55.9181" y2="50.7619" width="0.1524" layer="1"/>
 <wire x1="59.6519" y1="45.6946" x2="55.9181" y2="49.4284" width="0.1524" layer="1"/>
@@
 <wire x1="56.8071" y1="9.5123" x2="67.4624" y2="20.1676" width="0.1524" layer="1"/>
 <wire x1="52.7304" y1="9.5123" x2="56.8071" y2="9.5123" width="0.1524" layer="1"/>
-<wire x1="49.0601" y1="13.1826" x2="52.7304" y2="9.5123" width="0.1524" layer="1"/>
-<wire x1="49.0601" y1="13.1826" x2="49.022" y2="13.2207" width="0.1524" layer="16"/>
-<wire x1="49.022" y1="13.2207" x2="47.4472" y2="13.2207" width="0.1524" layer="16"/>
-<wire x1="46.7614" y1="12.5349" x2="47.4472" y2="13.2207" width="0.1524" layer="16"/>
-<wire x1="46.228" y1="12.5349" x2="46.7614" y2="12.5349" width="0.1524" layer="16"/>
+<wire x1="51.7271" y1="10.5156" x2="52.7304" y2="9.5123" width="0.1524" layer="1"/>
 <wire x1="55.9181" y1="50.7619" x2="55.88" y2="50.8" width="0.1524" layer="1"/>
-<via x="49.0601" y="13.1826" extent="1-16" drill="0.3048"/>
-<wire x1="46.228" y1="12.462" x2="43.704" y2="14.986" width="0.1524" layer="16"/>
-<wire x1="43.704" y1="14.986" x2="43.688" y2="14.986" width="0.1524" layer="16"/>
-<wire x1="43.688" y1="14.986" x2="43.307" y2="15.367" width="0.1524" layer="16"/>
-<wire x1="43.307" y1="15.367" x2="43.307" y2="15.4686" width="0.1524" layer="16"/>
-<via x="43.307" y="15.4686" extent="1-16" drill="0.35"/>
-<wire x1="46.228" y1="12.5349" x2="46.228" y2="12.462" width="0.1524" layer="16"/>
+<via x="51.7271" y="10.5156" extent="1-16" drill="0.3048"/>
+<via x="38.227" y="15.4686" extent="1-16" drill="0.35"/>
 <wire x1="18.97" y1="28.592" x2="19.1135" y2="28.4485" width="0.1524" layer="1"/>
 <wire x1="19.1135" y1="28.4485" x2="19.1135" y2="27.9019" width="0.1524" layer="1"/>
+<contactref element="D1" pad="1"/>
+<wire x1="38.227" y1="15.4686" x2="43.0276" y2="10.668" width="0.1524" layer="16"/>
+<via x="43.18" y="10.668" extent="1-16" drill="0.35"/>
+<wire x1="43.18" y1="10.668" x2="43.386" y2="10.462" width="0.1524" layer="1"/>
+<wire x1="43.386" y1="10.462" x2="46.228" y2="10.462" width="0.1524" layer="1"/>
+<wire x1="43.0276" y1="10.668" x2="43.18" y2="10.668" width="0.1524" layer="16"/>
+<wire x1="46.228" y1="10.462" x2="51.6735" y2="10.462" width="0.1524" layer="16"/>
+<wire x1="51.6735" y1="10.462" x2="51.7271" y2="10.5156" width="0.1524" layer="16"/>
 </signal>
 <signal name="IO27">
@@
 <contactref element="U3" pad="3"/>
 <contactref element="U1" pad="11"/>
-<contactref element="D1" pad="1"/>
 <wire x1="19.6977" y1="30.6959" x2="20.2311" y2="30.1625" width="0.1524" layer="1"/>
 <wire x1="18.9865" y1="30.6959" x2="19.6977" y2="30.6959" width="0.1524" layer="1"/>
@@
 <wire x1="17.4498" y1="23.5712" x2="16.7386" y2="24.2824" width="0.1524" layer="16"/>
 <wire x1="32.258" y1="23.5712" x2="17.4498" y2="23.5712" width="0.1524" layer="16"/>
-<wire x1="45.1612" y1="10.668" x2="40.76065" y2="15.06855" width="0.1524" layer="16"/>
+<wire x1="40.76065" y1="15.06855" x2="43.3832" y2="12.446" width="0.1524" layer="16"/>
 <wire x1="40.76065" y1="15.06855" x2="32.258" y2="23.5712" width="0.1524" layer="16"/>
-<wire x1="46.0502" y1="10.668" x2="45.1612" y2="10.668" width="0.1524" layer="16"/>
-<wire x1="46.228" y1="10.4902" x2="46.0502" y2="10.668" width="0.1524" layer="16"/>
-<wire x1="46.228" y1="10.4902" x2="46.228" y2="10.462" width="0.1524" layer="16"/>
 <wire x1="54.3306" y1="46.5582" x2="58.3438" y2="50.5714" width="0.1524" layer="16"/>
 <wire x1="53.1876" y1="45.4152" x2="54.3306" y2="46.5582" width="0.1524" layer="1"/>
@@
 <wire x1="20.2311" y1="30.1625" x2="20.2311" y2="28.6009" width="0.1524" layer="1"/>
 <wire x1="20.2311" y1="28.6009" x2="20.24" y2="28.592" width="0.1524" layer="1"/>
+<contactref element="D1" pad="2"/>
+<wire x1="46.212" y1="12.446" x2="46.228" y2="12.462" width="0.1524" layer="16"/>
+<wire x1="43.3832" y1="12.446" x2="46.212" y2="12.446" width="0.1524" layer="16"/>
 </signal>
 <signal name="IO14">
